Commit message: mesh import box

File: data/urdf/test_minimal.urdf (robot description, URDF)
Before this commit: robot test_minimal, 3 links, 2 joints
Links:
- link link1: geometry collision mesh filename=package://nao_model/mesh/dae/Torso.dae; visual box size=0.1 0.2 0.1
- link link2: geometry collision mesh filename=package://nao_model/mesh/dae/Torso.dae; visual box size=0.05 0.05 0.1

Commit message: Import mesh

File: data/urdf/test_minimal.urdf (robot description, URDF)
Before this commit: robot test_minimal, 3 links, 2 joints
Links:
- link base_link: geometry visual mesh filename=/home/nngoc/blender-urdf/data/mesh/atrv.stl

Commit message: import box, sphere, cyl, mesh

File: data/urdf/test_minimal.urdf (robot description, URDF)
Before this commit: robot test_minimal, 3 links, 2 joints
Links:
- link link1: geometry collision cylinder length=1 radius=0.1; visual box size=0.1 0.2 0.1
- link link2: geometry collision sphere radius=0.1; visual box size=0.05 0.05 0.1

Commit message: import plane mesh: ok

File: data/urdf/test_minimal.urdf (robot description, URDF)
Before this commit: robot test_minimal, 3 links, 2 joints
Links:
- link base_link: geometry visual mesh filename=/home/nngoc//miror_workspace/miror/miror_description/meshes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

Commit message: Update test_minimal.urdf to import box, cylinder, sphere, mesh

File: data/urdf/test_minimal.urdf (robot description, URDF)
Before this commit: robot test_minimal, 3 links, 2 joints
Links:
- link base_link: geometry visual mesh filename=/home/nngoc//miror_workspace/miror/miror_description/meshes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
- link link1: geometry collision cylinder length=1 radius=0.1; visual box size=0.1 0.2 0.1
- link link2: geometry collision sphere radius=0.1; visual box size=0.05 0.05 0.1

Commit message: temp

File: data/urdf/test_minimal.urdf (robot description, URDF)
Before this commit: robot test_minimal, 3 links, 2 joints
Links:
- link base_link: geometry visual mesh filename=/home/nngoc/miror_workspace/miror/miror_description/meshes/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
